File: PCB/FaikoutETH/Faikout.kicad_pcb (KiCad board)
At the start: 2 copper layers, 70 x 70 mm, 72 parts, among them J1 1x5, J2 TC2030-USB-NL, J3 Reset, J4 RJ45_LED, Q1 BSS138PS, U2 KSZ8851SNL, U4 ESP32-S3-MINI-1, U5 TPS62933, Y1 Crystal_GND24

Commit message: ETH board
Other:
- board text added: "DO NOT USE WITH X403"
- board text added: "Not certified for grid power saftey isolation"
- board text added: "Prototype/dev board for specialist/hobbyist use"

Commit message: New ETH
Parts:
- removed R13, R14: 49R9, RevK:R_0201
- removed U2: KSZ8851SNL, RevK:QFN-32-1EP_5x5mm_P0.5mm_EP3.7x3.7mm
- added U1: KSZ8851SNL, RevK:QFN-32-1EP_5x5mm_P0.5mm_EP3.7x3.7mm, F.Cu at (127.7, 73.0)
- J4: footprint RevK:HC-WK88-H21-DKH -> RevK:RC01516
- moved J4 12.5 mm to (151.7, 73.0)
- moved TR1 7.03 mm to (137.2, 73.0)
- moved C23 6.75 mm to (125.6, 81.0)
- moved C10 6.74 mm to (126.7, 79.2)
- moved C12 6.74 mm to (129.1, 79.6)
- moved C14 6.74 mm to (131.1, 69.1)
- moved C20 6.74 mm to (129.7, 65.4)
- moved C24 6.74 mm to (130.8, 67.7)
- moved C26 6.74 mm to (125.3, 68.6)
- moved C27 6.74 mm to (128.1, 65.8)
- moved C28 6.74 mm to (130.8, 68.3)
- moved C8 6.74 mm to (126.0, 79.8)
- moved D5 6.74 mm to (131.7, 65.6)
- moved D6 6.74 mm to (130.6, 65.6)
- moved R11 6.74 mm to (131.1, 70.2)
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Routing:
- net LED1: track 65.1 -> 0.00 mm, vias 1 -> 0
- net LED0: track 52.2 -> 0.00 mm, vias 1 -> 0
- net Net-(J4-Pad9): track 18.9 -> 0.00 mm, vias 1 -> 0
- net SH: track 15.7 -> 0.00 mm
- net Net-(J4-Pad11): track 7.03 -> 0.00 mm, vias 1 -> 0
- net SO: track 33.7 -> 27.2 mm
- net SCLK: track 31.5 -> 25.1 mm
- net CSN: track 25.5 -> 19.1 mm
- net SI: track 35.8 -> 29.8 mm
- net INTR: track 38.3 -> 32.3 mm
- net PME: track 37.6 -> 31.7 mm
- net GND: track 28.3 -> 34.2 mm, vias 93 -> 91
- net ETHRST: track 11.1 -> 5.30 mm, vias 2 -> 0
- net unconnected-(U1-LED1-Pad32): track 0.00 -> 4.53 mm, vias 0 -> 1
- net Net-(TR1-RD+): track 8.36 -> 5.66 mm
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- removed copper zone on B.Cu, net SH
- removed copper zone on F.Cu, net SH
Other:
- board text added: "Prototype/dev board for hobbyist use"
- board text removed: "Prototype/dev board for specialist/hobbyist use"
