File: PCB/FaikoutETH/Faikout.kicad_pcb (KiCad board)
At the start: 2 copper layers, 70 x 70 mm, 70 parts, among them J1 1x5, J2 TC2030-USB-NL, J3 Reset, J4 RJ45_LED, Q1 BSS138PS, U1 KSZ8851SNL, U4 ESP32-S3-MINI-1, U5 TPS62933, Y1 Crystal_GND24

Commit message: Tidy tracks
Parts:
- moved C10 0.70 mm to (126.1, 78.5)
Routing:
- net unconnected-(U1-LED1-Pad32): track 4.53 -> 0.00 mm, vias 1 -> 0
- net unconnected-(U1-LED0-Pad1): track 1.49 -> 0.00 mm, vias 1 -> 0
- net GND: vias 91 -> 90

Commit message: Re-render, latest layout
Other:
- board text added: "5 V-cuts"
- board text removed: "6 V-cuts"

Commit message: Extra GPIOs
Parts:
- added TP11: TestPoint, RevK:PAD-2mm, B.Cu at (125.5, 55.0)
- added TP12: TestPoint, RevK:PAD-2mm, B.Cu at (125.5, 52.8)
- added TP13: TestPoint, RevK:PAD-2mm, B.Cu at (125.5, 57.2)
- U1: footprint RevK:QFN-32-1EP_5x5mm_P0.5mm_EP3.7x3.7mm -> RevK:QFN-32-1EP_5x5mm_P0.5mm_EP3.7x3.7mm-hot
- moved TP6 4.50 mm to (130.9, 50.2)
- moved TP8 4.50 mm to (126.4, 50.2)
- moved J3 2.05 mm to (131.8, 55.0)
Connections:
- U4 pad 4: unconnected-(U4-GPIO0-Pad4) -> Net-(U4-GPIO0)
- U4 pad 5: unconnected-(U4-GPIO1-Pad5) -> Net-(U4-GPIO1)
- U4 pad 6: unconnected-(U4-GPIO2-Pad6) -> Net-(U4-GPIO2)
Routing:
- net Net-(U4-GPIO2): track 0.00 -> 10.4 mm, vias 0 -> 1
- net Net-(U4-GPIO1): track 0.00 -> 7.78 mm, vias 0 -> 1
- net Net-(U4-GPIO0): track 0.00 -> 5.19 mm, vias 0 -> 1
- net +3.3V: track 98.0 -> 100.1 mm
- net Net-(J3-Pin_2): track 7.10 -> 5.07 mm
- net D-: track 35.8 -> 34.5 mm
- net RST: track 20.3 -> 19.3 mm
- net GND: vias 90 -> 91
Other:
- board text added: "0"
- board text added: "2"
