File: PCB/FaikoutETH/Faikout.kicad_sch (KiCad schematic)
At the start: 71 parts, among them J1 1x5, J2 TC2030-USB-NL, J3 Reset, J4 RJ45_LED, Q1 BSS138PS, U2 KSZ8851SNL, U4 ESP32-S3-MINI-1, U5 TPS62933, Y1 Crystal_GND24

Commit message: Ethernet board
Parts:
- added V7: (no value), RevK:VCUT70N, symbol RevK:VCUT
- U2: footprint Package_DFN_QFN:QFN-32-1EP_5x5mm_P0.5mm_EP3.7x3.7mm -> RevK:QFN-32-1EP_5x5mm_P0.5mm_EP3.7x3.7mm
Connections:
- net CSN: now also U4.14 (GPIO10)
- net GND: no longer U4.16 (GPIO12), U4.17 (GPIO13), U4.18 (GPIO14), U4.19 (GPIO15), U4.20 (GPIO16)
- net INTR: now also U4.19 (GPIO15)
- net PME: now also U4.18 (GPIO14)
- net RST: no longer D5.1 (K)
- net SCLK: now also U4.16 (GPIO12)
- net SI: now also U4.15 (GPIO11)
- net SO: now also U4.17 (GPIO13)
- net ETHRST: now reaches U4.13 (GPIO9)
- net ETHRST: now also D5.1 (K)
- net VA1: no longer names the net of TR1.2 (C_TD)
- net VA2: no longer names the net of TR1.7 (C_RD)
- new net SH: J4.13 (SH), J4.14 (SH)
- no-connect marks 29 -> 28
Other:
- moved on the sheet: C6, R3

Commit message: Library update
Parts:
- FB3, FB4, FB5: footprint Inductor_SMD:L_0603_1608Metric -> RevK:L_0603
Changed lines of the file:
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@@
 			)
 		)
-		(property "Footprint" "Inductor_SMD:L_0603_1608Metric"
+		(property "Footprint" "RevK:L_0603"
 			(at 156.972 106.68 90)
 			(hide yes)
@@
 			)
 		)
-		(property "Footprint" "Inductor_SMD:L_0603_1608Metric"
+		(property "Footprint" "RevK:L_0603"
 			(at 122.428 106.68 90)
 			(hide yes)
@@
 			)
 		)
-		(property "Footprint" "Inductor_SMD:L_0603_1608Metric"
+		(property "Footprint" "RevK:L_0603"
 			(at 171.45 37.338 90)
 			(hide yes)

Commit message: ETH board
Parts:
- removed U2: KSZ8851SNL, RevK:QFN-32-1EP_5x5mm_P0.5mm_EP3.7x3.7mm, symbol RevK:KSZ8851SNL
Changed lines of the file:
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@@
 		(color 0 0 0 0)
 	)
-	(junction
-		(at 130.81 92.71)
-		(diameter 0)
-		(color 0 0 0 0)
-	)
 	(no_connect
 		(at 67.31 53.34)
@@
 		(in_bom no)
 		(on_board yes)
-		(in_pos_files yes)
+		(in_pos_files no)
 		(dnp no)
 		(fields_autoplaced yes)
@@
 	)
 	(symbol
-		(lib_id "RevK:KSZ8851SNL")
-		(at 139.7 71.12 0)
-		(unit 1)
-		(body_style 1)
-		(exclude_from_sim no)
-		(in_bom yes)
-		(on_board yes)
-		(in_pos_files yes)
-		(dnp no)
-		(property "Reference" "U2"
-			(at 139.954 69.85 0)
-			(show_name no)
-			(do_not_autoplace no)
-			(effects
-				(font
-					(size 1.27 1.27)
-				)
-			)
-		)
-		(property "Value" "KSZ8851SNL"
-			(at 139.954 72.39 0)
-			(show_name no)
-			(do_not_autoplace no)
-			(effects
-				(font
-					(size 1.27 1.27)
-				)
-			)
-		)
-		(property "Footprint" "RevK:QFN-32-1EP_5x5mm_P0.5mm_EP3.7x3.7mm"
-			(at 139.446 36.068 0)
-			(hide yes)
-			(show_name no)
-			(do_not_autoplace no)
-			(effects
-				(font
-					(size 1.27 1.27)
-				)
-			)
-		)
-		(property "Datasheet" "https://ww1.microchip.com/downloads/aemDocuments/documents/UNG/ProductDocuments/DataSheets/KSZ8851SNL-Single-Port-Ethernet-Controller-with-SPI-DS00002381C.pdf"
-			(at 139.192 36.322 0)
-			(hide yes)
-			(show_name no)
-			(do_not_autoplace no)
-			(effects
-				(font
-					(size 1.27 1.27)
-				)
-			)
-		)
-		(property "Description" "Single-Port Ethernet Controller with SPI"
-			(at 139.446 36.068 0)
-			(hide yes)
-			(show_name no)
-			(do_not_autoplace no)
-			(effects
-				(font
-					(size 1.27 1.27)
-				)
-			)
-		)
-		(pin "13"
-		)
-		(pin "12"
-		)
-		(pin "3"
-		)
-		(pin "2"
-		)
-		(pin "1"
-		)
-		(pin "7"
-		)
-		(pin "8"
-		)
-		(pin "4"
-		)
-		(pin "5"
-		)
-		(pin "20"
-		)
-		(pin "30"
-		)
-		(pin "31"
-		)
-		(pin "32"
-		)
-		(pin "10"
-		)
-		(pin "9"
-		)
-		(pin "17"
-		)
-		(pin "16"
-		)
-		(pin "15"
-		)
-		(pin "14"
-		)
-		(pin "19"
-		)
-		(pin "18"
-		)
-		(pin "21"
-		)
-		(pin "22"
-		)
-		(pin "25"
-		)
-		(pin "23"
-		)
-		(pin "24"
-		)
-		(pin "11"
-		)
-		(pin "6"
-		)
-		(pin "28"
-		)
-		(pin "29"
-		)
-		(pin "26"
-		)
-		(pin "27"
-		)
-		(pin "33"
-		)
-		(instances
-			(project "Faikout"
-				(path "/46c350bb-7de4-4e81-aafd-4af55e37aab0"
-					(reference "U2")
-					(unit 1)
-				)
-			)
-		)
-	)
-	(symbol
 		(lib_id "power:+1V8")
 		(at 101.6 110.49 90)
@@
 		(in_bom no)
 		(on_board yes)
-		(in_pos_files yes)
+		(in_pos_files no)
 		(dnp no)
 		(fields_autoplaced yes)
@@
 		(in_bom no)
 		(on_board yes)
-		(in_pos_files yes)
+		(in_pos_files no)
 		(dnp no)
 		(fields_autoplaced yes)
@@
 		(in_bom no)
 		(on_board yes)
-		(in_pos_files yes)
+		(in_pos_files no)
 		(dnp no)
 		(fields_autoplaced yes)
@@
 		(in_bom no)
 		(on_board yes)
-		(in_pos_files yes)
+		(in_pos_files no)
 		(dnp no)
 		(fields_autoplaced yes)
@@
 		(in_bom no)
 		(on_board yes)
-		(in_pos_files yes)
+		(in_pos_files no)
 		(dnp no)
 		(property "Reference" "PCB1"
@@
 		(in_bom no)
 		(on_board yes)
-		(in_pos_files yes)
+		(in_pos_files no)
 		(dnp no)
 		(fields_autoplaced yes)

Commit message: Added POE (not finished)
Parts:
- added U1: KSZ8851SNL, RevK:QFN-32-1EP_5x5mm_P0.5mm_EP3.7x3.7mm, symbol RevK:KSZ8851SNL
Connections:
- net +1V8: now also U1.23 (VDDD1V8), U1.5 (VDDCO1V8)
- net CSN: now also U1.26 (CSN)
- net GND: now also U1.13 (AGND), U1.18 (AGND), U1.22 (DGND), U1.24 (DGND), U1.29 (DGND), U1.33 (GND), U1.4 (DGND), U1.8 (AGND)
- net INTR: now also U1.3 (INTR)
- net LED0: now also U1.1 (LED0)
- net LED1: now also U1.32 (LED1)
- net PME: now also U1.2 (PME)
- net RSTN: now also U1.19 (RSTN)
- net RXN: now also U1.12 (RXN)
- net RXP: now also U1.11 (RXP)
- net SCLK: now also U1.28 (SCLK)
- net SI: now also U1.31 (SI)
- net SO: now also U1.27 (SO)
- net TXN: now also U1.15 (TXN)
- net TXP: now also U1.14 (TXP)
- net VDDA3V3: now also U1.16 (VDDA3V3)
- net VDDIO: now also U1.25 (VDDIO), U1.30 (VDDIO)
- net at C11.1, C12.1, FB3.2: now also U1.9 (VDDA1V8)
- net at R12.2: now also U1.17 (ISET)
- net at C27.1, Y1.3: now also U1.20 (X1)
- net at C26.1, Y1.1: now also U1.21 (X2)
Changed lines of the file:
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@@
 	)
 	(junction
+		(at 130.81 92.71)
+		(diameter 0)
+		(color 0 0 0 0)
+	)
+	(junction
 		(at 163.83 87.63)
 		(diameter 0)
@@
 					(unit 1)
 				)
+			)
+		)
+	)
+	(symbol
+		(lib_id "RevK:KSZ8851SNL")
+		(at 139.7 71.12 0)
+		(unit 1)
+		(body_style 1)
+		(exclude_from_sim no)
+		(in_bom yes)
+		(on_board yes)
+		(in_pos_files yes)
+		(dnp no)
+		(property "Reference" "U1"
+			(at 139.954 69.85 0)
+			(show_name no)
+			(do_not_autoplace no)
+			(effects
+				(font
+					(size 1.27 1.27)
+				)
+			)
+		)
+		(property "Value" "KSZ8851SNL"
+			(at 139.954 72.39 0)
+			(show_name no)
+			(do_not_autoplace no)
+			(effects
+				(font
+					(size 1.27 1.27)
+				)
+			)
+		)
+		(property "Footprint" "RevK:QFN-32-1EP_5x5mm_P0.5mm_EP3.7x3.7mm"
+			(at 139.446 36.068 0)
+			(hide yes)
+			(show_name no)
+			(do_not_autoplace no)
+			(effects
+				(font
+					(size 1.27 1.27)
+				)
+			)
+		)
+		(property "Datasheet" "https://ww1.microchip.com/downloads/aemDocuments/documents/UNG/ProductDocuments/DataSheets/KSZ8851SNL-Single-Port-Ethernet-Controller-with-SPI-DS00002381C.pdf"
+			(at 139.192 36.322 0)
+			(hide yes)
+			(show_name no)
+			(do_not_autoplace no)
+			(effects
+				(font
+					(size 1.27 1.27)
+				)
+			)
+		)
+		(property "Description" "Single-Port Ethernet Controller with SPI"
+			(at 139.446 36.068 0)
+			(hide yes)
+			(show_name no)
+			(do_not_autoplace no)
+			(effects
+				(font
+					(size 1.27 1.27)
+				)
+			)
+		)
+		(property "Rotation Offset" "90"
+			(at 139.7 71.12 0)
+			(hide yes)
+			(show_name no)
+			(do_not_autoplace no)
+			(effects
+				(font
+					(size 1.27 1.27)
+				)
+			)
+		)
+		(property "MPN" "C633272"
+			(at 139.7 71.12 0)
+			(hide yes)
+			(show_name no)
+			(do_not_autoplace no)
+			(effects
+				(font
+					(size 1.27 1.27)
+				)
+			)
+		)
+		(pin "13"
+		)
+		(pin "12"
+		)
+		(pin "3"
+		)
+		(pin "2"
+		)
+		(pin "1"
+		)
+		(pin "7"
+		)
+		(pin "8"
+		)
+		(pin "4"
+		)
+		(pin "5"
+		)
+		(pin "20"
+		)
+		(pin "30"
+		)
+		(pin "31"
+		)
+		(pin "32"
+		)
+		(pin "10"
+		)
+		(pin "9"
+		)
+		(pin "17"
+		)
+		(pin "16"
+		)
+		(pin "15"
+		)
+		(pin "14"
+		)
+		(pin "19"
+		)
+		(pin "18"
+		)
+		(pin "21"
+		)
+		(pin "22"
+		)
+		(pin "25"
+		)
+		(pin "23"
+		)
+		(pin "24"
+		)
+		(pin "11"
+		)
+		(pin "6"
+		)
+		(pin "28"
+		)
+		(pin "29"
+		)
+		(pin "26"
+		)
+		(pin "27"
+		)
+		(pin "33"
+		)
+		(instances
+			(project "Faikout"
+				(path "/46c350bb-7de4-4e81-aafd-4af55e37aab0"
+					(reference "U1")
+					(unit 1)
+				)

Commit message: New ETH
Parts:
- removed R13, R14: 49R9, RevK:R_0201, symbol Device:R
- J4: footprint RevK:HC-WK88-H21-DKH -> RevK:RC01516; symbol RevK:HC-WK88-H21-DKH -> RevK:RC01516; MPN C48618190 -> C708636; Position Offset (none) -> 0,0.5
Connections:
- net LED0: no longer names the net of U1.1 (LED0)
- net LED0: no longer J4.12
- net LED1: no longer names the net of U1.32 (LED1)
- net LED1: no longer J4.10
- removed net SH: J4.13 (SH), J4.14 (SH)
- no-connect marks 28 -> 30

Commit message: Tidy
Parts:
- C6: MPN (none) -> C87143
- R1, R17, R2, R3, R7: MPN C106225 -> C138117
Changed lines of the file:
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@@
 			)
 		)
-		(property "Sim.Enable" "0"
-			(at 262.255 170.815 0)
-			(hide yes)
-			(show_name no)
-			(do_not_autoplace no)
-			(effects
-				(font
-					(size 1.27 1.27)
-				)
-			)
-		)
 		(instances
 			(project "Faikout"
@@
 			)
 		)
-		(property "MPN" "C106225"
+		(property "MPN" "C138117"
 			(at 107.95 167.64 0)
 			(hide yes)
@@
 			)
 		)
-		(property "Sim.Enable" "0"
-			(at 259.08 173.99 0)
-			(hide yes)
-			(show_name no)
-			(do_not_autoplace no)
-			(effects
-				(font
-					(size 1.27 1.27)
-				)
-			)
-		)
 		(instances
 			(project "Faikout"
@@
 			)
 		)
-		(property "Sim.Enable" "0"
-			(at 262.255 177.165 0)
-			(hide yes)
-			(show_name no)
-			(do_not_autoplace no)
-			(effects
-				(font
-					(size 1.27 1.27)
-				)
-			)
-		)
 		(instances
 			(project "Faikout"
@@
 			)
 		)
-		(property "Sim.Enable" "0"
-			(at 260.35 173.99 0)
-			(hide yes)
-			(show_name no)
-			(do_not_autoplace no)
-			(effects
-				(font
-					(size 1.27 1.27)
-				)
-			)
-		)
 		(instances
 			(project "Faikout"
@@
 			)
 		)
-		(property "Sim.Enable" "0"
-			(at 265.43 173.99 0)
-			(hide yes)
-			(show_name no)
-			(do_not_autoplace no)
-			(effects
-				(font
-					(size 1.27 1.27)
-				)
-			)
-		)
 		(instances
 			(project "Faikout"
@@
 			)
 		)
-		(property "MPN" "C106225"
+		(property "MPN" "C138117"
 			(at 232.41 105.41 90)
 			(hide yes)
@@
 			)
 		)
-		(property "MPN" "C106225"
+		(property "MPN" "C138117"
 			(at 109.22 34.29 90)
 			(hide yes)
@@
 			)
 		)
-		(property "MPN" "C106225"
+		(property "MPN" "C138117"
 			(at 207.01 111.125 90)
 			(hide yes)
@@
 			)
 		)
+		(property "MPN" "C87143"
+			(at 76.2 81.28 0)
+			(hide yes)
+			(show_name no)
+			(do_not_autoplace no)
+			(effects
+				(font
+					(size 1.27 1.27)
+				)
+			)
+		)
 		(pin "1"
 		)
@@
 			)
 		)
-		(property "MPN" "C106225"
+		(property "MPN" "C138117"
 			(at 76.2 73.66 90)
 			(hide yes)
