File: PCB/FaikoutETH/Faikout.kicad_sch (KiCad schematic)
At the start: 70 parts, among them J1 1x5, J2 TC2030-USB-NL, J3 Reset, J4 RJ45_LED, Q1 BSS138PS, U1 KSZ8851SNL, U4 ESP32-S3-MINI-1, U5 TPS62933, Y1 Crystal_GND24

Commit message: Tidy tracks
Parts:
- U1: Rotation Offset 90 -> -90
Changed lines of the file:
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@@
 			)
 		)
-		(property "Rotation Offset" "90"
+		(property "Rotation Offset" "-90"
 			(at 139.7 71.12 0)
 			(hide yes)

Commit message: Extra GPIOs
Parts:
- added TP11, TP12, TP13: TestPoint, RevK:PAD-2mm, symbol Connector:TestPoint
- U1: footprint RevK:QFN-32-1EP_5x5mm_P0.5mm_EP3.7x3.7mm -> RevK:QFN-32-1EP_5x5mm_P0.5mm_EP3.7x3.7mm-hot
Connections:
- net GND: now also J4.S
- net at U4.4 (GPIO0): now also TP13.1
- net at U4.5 (GPIO1): now also TP11.1
- net at U4.6 (GPIO2): now also TP12.1
- no-connect marks 30 -> 27
