File: PCB/FaikoutETH/Faikout.kicad_sch (KiCad schematic)
At the start: 73 parts, among them J1 1x5, J2 TC2030-USB-NL, J3 Reset, J4 RJ45_LED, Q1 BSS138PS, U1 KSZ8851SNL, U4 ESP32-S3-MINI-1, U5 TPS62933, Y1 Crystal_GND24

Commit message: Tweak RJ45
Parts:
- J4: Position Offset 0,0.5 -> 0,0.4
Changed lines of the file:
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@@
 			)
 		)
-		(property "Position Offset" "0,0.5"
+		(property "Position Offset" "0,0.4"
 			(at 210.82 34.29 0)
 			(hide yes)

Commit message: New inductor
Parts:
- removed C29: 10uF 35V, RevK:C_0603, symbol Device:C
- removed C30, C32: 100nF 35V, RevK:C_0201, symbol Device:C
- removed C31: 33nF, RevK:C_0201, symbol Device:C
- removed C33: 100uF 6.3V, RevK:C_0805, symbol Device:C
- removed L13: 4.7uH, RevK:L_5x5, symbol Device:L
- removed R15: 33k, RevK:R_0201, symbol Device:R
- removed R16: 30.9k 1%, RevK:R_0201, symbol Device:R
- removed R17: 10k, RevK:R_0201, symbol Device:R
- removed U5: TPS62933, RevK:SOT-583-8, symbol Regulator_Switching:TPS62933
- added C1: 10uF 35V, RevK:C_0603, symbol Device:C
- added C2, C4: 100nF 35V, RevK:C_0201, symbol Device:C
- added C3: 33nF, RevK:C_0201, symbol Device:C
- added C5: 100uF 6.3V, RevK:C_0805, symbol Device:C
- added L1: 4.7uH, RevK:L_6x6, symbol Device:L
- added R5: 33k, RevK:R_0201, symbol Device:R
- added R6: 30.9k 1%, RevK:R_0201, symbol Device:R
- added R8: 10k, RevK:R_0201, symbol Device:R
- added U2: TPS62933, RevK:SOT-583-8, symbol Regulator_Switching:TPS62933
- U1: footprint RevK:QFN-32-1EP_5x5mm_P0.5mm_EP3.7x3.7mm-hot -> RevK:QFN-32-1EP_5x5mm_P0.5mm_EP3.7x3.7mm
- Y1: footprint Crystal:Crystal_SMD_3225-4Pin_3.2x2.5mm -> RevK:Crystal-3.2x2.5
Connections:
- net +3.3V: now also C5.1, L1.2, R6.1
- net BST: now also C4.1, U2.6 (BST)
- net DC: now also C1.1, C2.1, U2.3 (VIN)
- net FB: now also R6.2, R8.1, U2.8 (FB)
- net GND: now also C1.2, C2.2, C3.2, C5.2, R5.2, R8.2, U2.4 (GND)
- net RT: now also R5.1, U2.1 (RT)
- net SS: now also C3.1, U2.7 (SS)
- net SW: now also C4.2, L1.1, U2.5 (SW)

Commit message: Tweaks
Parts:
- U1: footprint RevK:QFN-32-1EP_5x5mm_P0.5mm_EP3.7x3.7mm -> RevK:QFN-32-1EP_5x5mm_P0.5mm_EP3.7x3.7mm-hot
- Y1: Rotation Offset (none) -> 180
Changed lines of the file:
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@@
 			)
 		)
+		(property "Rotation Offset" "180"
+			(at 176.53 71.12 90)
+			(hide yes)
+			(show_name no)
+			(do_not_autoplace no)
+			(effects
+				(font
+					(size 1.27 1.27)
+				)
+			)
+		)
 		(pin "4"
 		)
@@
 			)
 		)
-		(property "Footprint" "RevK:QFN-32-1EP_5x5mm_P0.5mm_EP3.7x3.7mm"
+		(property "Footprint" "RevK:QFN-32-1EP_5x5mm_P0.5mm_EP3.7x3.7mm-hot"
 			(at 139.446 36.068 0)
 			(hide yes)
