File: PCB/FaikoutPOE/Faikout.kicad_pcb (KiCad board)
At the start: 2 copper layers, 58 x 65 mm, 85 parts, among them J1 RJ45_LED, J2 S21, J5 Reset, J7 TC2030-USB-NL-DS, M3 Ag97012-FL, P1 Square, Q1 BSS138PS, U1 KSZ8851SNL, U2 ESP32-S3-MINI-1, U3 TCMT1100, U4 TPS62933, U5 TCMT1100, Y1 Crystal_GND24

Commit message: Started on POE
Parts:
- removed C35: 100nF, RevK:C_0201
- removed D21: DKS34, RevK:D_SOD-123FL
- added D3: ~, RevK:DFN1006-2L, F.Cu at (131.9, 66.0)
- D5: value XL-1615RGBC-2812B -> ~; footprint RevK:SMD1615-Side -> RevK:DFN1006-2L
- D6, D7: value XL-1615RGBC-2812B -> D; footprint RevK:SMD1615-Side -> RevK:D_0402
- J1: footprint RevK:HC-WK88-H21-DKH -> RevK:RC01516
- P1: moved to B.Cu
- R6: value 49R9 -> 10k
- moved C36 48.0 mm to (117.8, 89.5)
- moved R9 48.0 mm to (117.8, 90.5)
- moved C34 42.9 mm to (119.8, 87.2)
- moved D4 42.9 mm to (119.3, 85.7)
- moved C17 41.9 mm to (116.0, 85.2)
- moved D6 35.3 mm to (132.0, 69.5)
- moved D7 34.7 mm to (133.3, 67.8), turned to -90 degrees
- moved R18 32.4 mm to (119.9, 89.0)
- moved R19 32.4 mm to (119.3, 89.0)
- moved J7 29.4 mm to (123.0, 90.5), turned to 180 degrees
- moved R5 27.7 mm to (125.2, 65.6)
- moved J2 26.3 mm to (136.5, 71.0), turned to 0 degrees
- moved U2 26.0 mm to (108.5, 73.5)
- moved P1 25.7 mm to (103.0, 72.0), turned to 180 degrees
- moved J5 25.6 mm to (108.5, 73.5)
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Connections:
- C29 pad 1: VDC -> POE
- C30 pad 1: VDC -> POE
- D4 pad 2: LED -> LEDO
- D4 pad 4: Net-(D4-O) -> LEDI
- D5 pad 1: GND -> S21GND
- D5 pad 2: Net-(D4-O) -> S21RX
- D6 pad 1: GND -> S21RX
- D6 pad 2: Net-(D5-O) -> Net-(D6-A)
- D7 pad 1: GND -> S21TX
- D7 pad 2: Net-(D6-O) -> Net-(D6-A)
- J2 pad 1: unconnected-(J2-Pin_1-Pad1) -> S215V
- J2 pad 2: unconnected-(J2-Pin_2-Pad2) -> S21RX
- J2 pad 3: unconnected-(J2-Pin_3-Pad3) -> S21TX
- J2 pad 5: unconnected-(J2-Pin_5-Pad5) -> S21GND
- R5 pad 2: Net-(J1-Pad11) -> Net-(R5-Pad2)
- R6 pad 1: +3.3V -> S215V
- R6 pad 2: Net-(J1-Pad9) -> Net-(D6-A)
- U1 pad 1: LED0 -> unconnected-(U1-LED0-Pad1)
- U1 pad 32: LED1 -> unconnected-(U1-LED1-Pad32)
- U2 pad 27: unconnected-(U2-GPIO47-Pad27) -> LEDO
- U2 pad 28: unconnected-(U2-GPIO33-Pad28) -> LEDI
- U2 pad 29: unconnected-(U2-GPIO34-Pad29) -> RX
- U2 pad 30: unconnected-(U2-GPIO48-Pad30) -> TX
- U2 pad 41: LEDI -> unconnected-(U2-GPIO45-Pad41)
- U2 pad 44: LED -> unconnected-(U2-GPIO46-Pad44)
- U3 pad 1: unconnected-(U3-Pad1) -> Net-(R5-Pad2)
- U3 pad 2: unconnected-(U3-Pad2) -> TX
- U3 pad 3: unconnected-(U3-Pad3) -> S21GND
- U3 pad 4: unconnected-(U3-Pad4) -> S21TX
- U4 pad 3: VDC -> POE
- U5 pad 1: unconnected-(U5-Pad1) -> S215V
- U5 pad 2: unconnected-(U5-Pad2) -> S21RX
- U5 pad 3: unconnected-(U5-Pad3) -> GND
- U5 pad 4: unconnected-(U5-Pad4) -> RX
Routing:
- net +3.3V: track 132.2 -> 0.00 mm, vias 4 -> 0
- net LEDI: track 75.8 -> 0.00 mm, vias 2 -> 0
- net LED1: track 68.8 -> 0.00 mm, vias 3 -> 0
- net VDC: track 61.0 -> 0.00 mm, vias 2 -> 0
- net LED: track 60.5 -> 0.00 mm, vias 2 -> 0
- net LED0: track 54.6 -> 0.00 mm, vias 3 -> 0
- net POELOAD: track 44.4 -> 0.00 mm, vias 2 -> 0
- net INTR: track 42.4 -> 0.00 mm, vias 2 -> 0
- net PME: track 41.6 -> 0.00 mm, vias 2 -> 0
- net ETHRST: track 35.3 -> 0.00 mm, vias 2 -> 0
- net SI: track 33.9 -> 0.00 mm, vias 2 -> 0
- net CSN: track 33.3 -> 0.00 mm, vias 2 -> 0
- net SCLK: track 30.1 -> 0.00 mm, vias 2 -> 0
- net SO: track 30.0 -> 0.00 mm, vias 2 -> 0
- net VDDA3V3: track 25.7 -> 0.60 mm
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- added copper zone on B.Cu, net S21GND
- added copper zone on F.Cu, net S21GND
- removed copper zone on B.Cu, net Net-(J1-SH-Pad13)
- removed copper zone on F.Cu, net Net-(J1-SH-Pad13)
Other:
- board size 58 x 65 mm -> 58 x 36 mm
- board text added: "Faikout ${CURRENT_DATE}"
- board text added: "S21"
- board text removed: "10 11 12 13 14 15 16 36 45 46"
- board text removed: "CSN MOSI SCLK MISO PME INTR ETHRST POELOAD LEDI LED"
- board text removed: "EnvLED2 ${CURRENT_DATE}"
- board text removed: "H"
- board text removed: "T3902"
- board text removed: "U"

Commit message: PoE layout, not tracked yet
Parts:
- added R10: 49R9, RevK:R_0201, F.Cu at (109.0, 79.6)
- moved D4 42.4 mm to (156.5, 65.5), turned to -90 degrees
- moved D3 33.5 mm to (102.2, 81.6), turned to -90 degrees
- moved R5 32.5 mm to (101.9, 88.3), turned to 0 degrees
- moved D7 31.8 mm to (104.0, 80.2), turned to 0 degrees
- moved U3 30.1 mm to (104.0, 85.0), turned to 90 degrees
- moved J2 29.8 mm to (107.3, 77.0), turned to 90 degrees
- moved D1 29.8 mm to (143.2, 64.9)
- moved C16 29.8 mm to (143.2, 65.5)
- moved FB5 29.8 mm to (145.7, 65.0), turned to 0 degrees
- moved D6 28.9 mm to (105.8, 81.5), turned to 90 degrees
- moved D5 27.6 mm to (107.2, 80.2), turned to 180 degrees
- moved D2 26.9 mm to (141.6, 65.1), turned to 90 degrees
- moved R7 26.6 mm to (140.9, 65.2), turned to 90 degrees
- moved C4 26.5 mm to (140.3, 65.2), turned to 90 degrees
- moved C3 26.4 mm to (139.7, 65.2), turned to 90 degrees
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Connections:
- U5 pad 2: S21RX -> Net-(R10-Pad1)
Routing:
- net E78: track 28.9 -> 0.00 mm, vias 3 -> 0
- net E36: track 24.4 -> 0.00 mm, vias 3 -> 0
- net GND: track 22.7 -> 0.00 mm, vias 30 -> 0
- net E12: track 17.0 -> 0.00 mm, vias 3 -> 0
- net E45: track 16.3 -> 0.00 mm, vias 3 -> 0
- net Net-(M3-VINC): track 15.7 -> 0.00 mm, vias 1 -> 0
- net Net-(M3-VINB): track 13.7 -> 0.00 mm
- net VDDIO: track 8.54 -> 0.00 mm
- net Net-(M3-VINA): track 8.38 -> 0.00 mm
- net Net-(M3-VIND): track 8.20 -> 0.00 mm
- net Net-(TR1-RD+): track 6.56 -> 0.00 mm
- net Net-(TR1-RD-): track 6.38 -> 0.00 mm
- net Net-(U1-X1): track 5.98 -> 0.00 mm
- net Net-(TR1-TD+): track 4.56 -> 0.00 mm
- net Net-(U1-VDDA1V8): track 4.53 -> 0.00 mm
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Other:
- outline, holes or cut-outs redrawn
- board text added: "5V input required"
- board text added: "A"
- board text added: "Not certified for grid power isolation"
- board text added: "Opto isolated"

Commit message: Tweaks
Parts:
- removed D6, D7: D, RevK:D_0402
- moved L10 0.60 mm to (142.2, 92.0)
- moved L11 0.60 mm to (145.1, 92.0)
- moved L12 0.60 mm to (148.0, 92.0)
Connections:
- R6 pad 2: Net-(D6-A) -> S21TX
- U5 pad 1: S215V -> Net-(R10-Pad1)
- U5 pad 2: Net-(R10-Pad1) -> S21GND
Routing:
- removed copper zone on F.Cu, net SW

Commit message: Tidy models
Parts:
- moved M3 49.7 mm to (105.6, 97.2), turned to 180 degrees
- moved F3 47.3 mm to (108.5, 44.6), turned to -90 degrees
- moved R5 45.4 mm to (111.7, 43.9), turned to -90 degrees
- moved D3 40.7 mm to (118.4, 44.2), turned to 180 degrees
- moved U3 40.6 mm to (115.0, 46.0), turned to 0 degrees
- moved L12 40.0 mm to (108.0, 90.0), turned to -90 degrees
- moved D4 39.7 mm to (134.5, 98.5), turned to 180 degrees
- moved R22 38.0 mm to (105.4, 58.1), turned to 180 degrees
- moved L11 37.4 mm to (108.0, 87.1), turned to -90 degrees
- moved R20 37.1 mm to (109.0, 54.0), turned to -90 degrees
- moved J1 37.0 mm to (117.5, 94.5), turned to 0 degrees
- moved U5 36.3 mm to (115.0, 49.5), turned to 180 degrees
- moved L9 36.0 mm to (105.6, 81.0), turned to -90 degrees
- moved Q1 35.8 mm to (106.2, 60.0), turned to 90 degrees
- moved L10 35.1 mm to (108.0, 84.2), turned to -90 degrees
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Other:
- board size 58 x 36 mm -> 36 x 58 mm

Commit message: Tweak design
Parts:
- removed C19: 100nF 35V, RevK:C_0201
- removed C20: 10uF 50V, RevK:C_1206
- removed C21: 100uF 50V, Capacitor_SMD:CP_Elec_6.3x7.7
- removed C23, C24: 10nF, RevK:C_0402
- removed D3: ~, RevK:DFN1006-2L
- removed F3: 1210L150/33WR, RevK:Fuse_1210
- removed J2: S21, RevK:JST_EH_S5B-EH_1x05_P2.50mm_Horizontal
- removed L1, L10, L11, L12, L2, L3, L4, L5, L6, L7, L8, L9: CBG201209U121T, RevK:L_0805
- removed M3: Ag97012-FL, RevK:Ag970XX-FL
- added C22: 100nF 35V, RevK:C_0201, F.Cu at (89.6, 77.1)
- added C25: 10uF 50V, RevK:C_1206, F.Cu at (91.2, 71.3)
- added C26: 100uF 50V, RevK:CP_Elec_6.3x7.7, F.Cu at (83.4, 71.0)
- added D11: ~, RevK:DFN1006-2L, F.Cu at (152.4, 56.3)
- added D21: DKS34, RevK:D_SOD-123FL, F.Cu at (91.4, 68.4)
- added D6: SMAJ58A, RevK:D_SMA, F.Cu at (81.4, 77.1)
- added D7: ~, RevK:DFN1006-2L, F.Cu at (152.4, 54.6)
- added D8: MB4S, RevK:TO-269AA-BR, F.Cu at (73.8, 70.1)
- added D9: MB4S, RevK:TO-269AA-BR, F.Cu at (73.8, 76.5)
- added F4: 1210L150/33WR, RevK:Fuse_1210, F.Cu at (91.2, 74.5)
- added J3: S21, RevK:JST_EH_S5B-EH_1x05_P2.50mm_Horizontal, F.Cu at (148.6, 51.8)
- added L14: CBG201209U121T, RevK:L_0805, F.Cu at (96.6, 52.1)
- added L15: CBG201209U121T, RevK:L_0805, F.Cu at (96.6, 54.4)
- added L16: CBG201209U121T, RevK:L_0805, F.Cu at (96.6, 56.6)
- added L17: CBG201209U121T, RevK:L_0805, F.Cu at (96.6, 58.9)
- added L18: CBG201209U121T, RevK:L_0805, F.Cu at (96.6, 61.1)
- added L19: CBG201209U121T, RevK:L_0805, F.Cu at (96.6, 63.4)
- added M1: Ag9912-LP, RevK:Ag9900-LP, F.Cu at (82.1, 58.5)
- added Q2: BSS138PS, RevK:SOT-363_SC-70-6, F.Cu at (149.5, 55.5)
- added R13: 10k, RevK:R_0201, F.Cu at (146.4, 56.0)
- added R16: 10k, RevK:R_0201, F.Cu at (146.4, 57.5)
- D5: value ~ -> D; footprint RevK:DFN1006-2L -> RevK:D_0402
- R10: value 49R9 -> 1k
- moved R6 37.5 mm to (156.3, 57.0)
- moved D5 35.6 mm to (155.0, 54.6), turned to 0 degrees
- moved R10 26.2 mm to (146.4, 54.5)
- moved TR1 1.00 mm to (117.4, 80.0)
Connections:
- net S21TX renamed Net-(Q2B-GP)
- C29 pad 1: POE -> VDC
- C30 pad 1: POE -> VDC
- D5 pad 1: S21GND -> Net-(D5-K)
- D5 pad 2: S21RX -> Net-(D5-A)
- R10 pad 1: Net-(R10-Pad1) -> S21DC
- R10 pad 2: S21RX -> Net-(R10-Pad2)
- R6 pad 1: S215V -> S21DC
- U4 pad 3: POE -> VDC
- U5 pad 1: Net-(R10-Pad1) -> Net-(R10-Pad2)
- U5 pad 2: S21GND -> Net-(Q2A-DN)
Other:
- board text removed: "Ag97012-FL for PoE"

Commit message: Started POE
Parts:
- Y1: footprint Crystal:Crystal_SMD_3225-4Pin_3.2x2.5mm -> RevK:Crystal-3.2x2.5
- moved D4 60.7 mm to (101.5, 47.5)
- moved C22 46.2 mm to (125.7, 48.2)
- moved Q2 45.9 mm to (106.4, 39.8)
- moved R6 44.0 mm to (115.2, 41.2)
- moved D11 44.0 mm to (111.4, 40.5)
- moved D7 44.0 mm to (111.4, 38.9)
- moved D5 43.8 mm to (113.5, 40.5)
- moved R16 40.8 mm to (109.4, 40.5)
- moved R10 40.6 mm to (109.4, 38.0)
- moved R13 40.6 mm to (109.4, 39.5)
- moved D8 38.7 mm to (104.5, 93.7)
- moved C26 36.1 mm to (113.8, 51.5), turned to 180 degrees
- moved J7 35.6 mm to (137.5, 49.0), turned to 0 degrees
- moved J3 35.4 mm to (115.9, 38.1)
- moved D9 32.7 mm to (104.5, 88.0)
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Connections:
- J1 pad S1: (no net) -> unconnected-(J1-PadS1)
- J1 pad S2: (no net) -> GND
- J7 pad 1: VBUS -> VDC
Routing:
- removed copper zone on B.Cu, net GND
- removed copper zone on F.Cu, net GND
- removed copper zone on B.Cu, net S21GND
- removed copper zone on F.Cu, net S21GND
Other:
- board size 36 x 58 mm -> 42 x 69 mm
- board text added: "Faikout PoE ${CURRENT_DATE}"
- board text removed: "5V input required"
- board text removed: "Faikout ${CURRENT_DATE}"

Commit message: Progress
Parts:
- moved Q2 20.6 mm to (127.0, 40.9), turned to 180 degrees
- moved D7 17.7 mm to (129.1, 38.9), turned to -90 degrees
- moved D11 17.6 mm to (129.0, 40.6), turned to 90 degrees
- moved R10 15.1 mm to (124.3, 40.5), turned to -90 degrees
- moved R6 9.78 mm to (125.0, 40.5), turned to -90 degrees
- moved R16 7.92 mm to (117.3, 40.0)
- moved R13 6.71 mm to (116.0, 40.8)
- moved D5 2.53 mm to (116.0, 40.0), turned to 180 degrees
- moved J3 0.08 mm to (116.0, 38.1)
Routing:
- net Net-(J3-Pin_3): track 0.00 -> 15.5 mm, vias 0 -> 2
- net Net-(Q2B-GP): track 0.00 -> 11.7 mm, vias 0 -> 2
- net Net-(Q2A-DN): track 0.00 -> 5.14 mm
- net Net-(J3-Pin_2): track 0.00 -> 3.38 mm
- net S21DC: track 0.00 -> 3.15 mm
- net Net-(D5-A): track 0.00 -> 2.93 mm
- net Net-(R10-Pad2): track 0.00 -> 1.08 mm
- net Net-(D5-K): track 0.00 -> 0.62 mm
- added copper zone on B.Cu, net S21GND
- added copper zone on F.Cu, net S21GND
Other:
- outline, holes or cut-outs redrawn
- board text added: "0V"
- board text added: "12V"
- board text added: "5V"
- board text added: "<"
- board text added: ">"
