File: PCB/FaikoutPOE/Faikout.kicad_pcb (KiCad board)
At the start: 2 copper layers, 42 x 69 mm, 83 parts, among them J1 RJ45_LED, J3 S21, J5 Reset, J7 TC2030-USB-NL-DS, M1 Ag9912-LP, P1 Square, Q1 BSS138PS, Q2 BSS138PS, U1 KSZ8851SNL, U2 ESP32-S3-MINI-1, U3 TCMT1100, U4 TPS62933, U5 TCMT1100, Y1 Crystal_GND24

Commit message: Tweak
Parts:
- added D10: D, RevK:D_0402, F.Cu at (114.7, 40.6)
- moved R10 0.60 mm to (124.3, 41.1)
- moved R6 0.60 mm to (125.0, 41.1)
Connections:
- D5 pad 2: Net-(D5-A) -> Net-(D10-A)
- J3 pad 1: Net-(D5-A) -> Net-(D10-A)
- R13 pad 1: Net-(D5-A) -> Net-(D10-K)
Routing:
- net Net-(D10-A): track 0.00 -> 3.20 mm
- net Net-(D5-A): track 2.93 -> 0.00 mm
- net Net-(D10-K): track 0.00 -> 1.09 mm
- net S21DC: track 3.15 -> 3.75 mm

Commit message: Tidy
Parts:
- added R17: 1k, RevK:R_0201, F.Cu at (122.3, 48.9)
- J7: moved to F.Cu
- moved U5 0.50 mm to (123.0, 44.0)
- moved R10 0.22 mm to (124.5, 41.1)
- moved R6 0.12 mm to (125.1, 41.1)
- turned J7 to 180 degrees
Routing:
- net VDC: track 24.0 -> 27.4 mm, vias 1 -> 2
- net Net-(D6-A2): track 18.0 -> 20.4 mm
- net RX: track 40.3 -> 41.3 mm
- net Net-(D6-A1): track 22.6 -> 21.7 mm
- net D-: track 29.1 -> 30.0 mm, vias 1 -> 2
- net +3.3V: track 141.2 -> 141.7 mm
- net D+: track 28.1 -> 28.3 mm, vias 1 -> 2
- net GND: vias 22 -> 61

Commit message: Re-render, latest layout
Parts:
- R20: value 220 1W -> 200 1W
- moved C6 1.23 mm to (140.0, 79.8), turned to 90 degrees
- moved D4 0.50 mm to (101.7, 48.0)
- moved Q1 0.50 mm to (105.0, 48.0)
- moved R21 0.50 mm to (106.9, 48.3)
- moved R22 0.50 mm to (103.2, 47.6)
- moved J7 0.49 mm to (137.5, 49.5)
- moved C7 0.23 mm to (140.7, 78.8), turned to 135 degrees
- moved FB3 0.10 mm to (140.9, 81.5)
Routing:
- net VDC: track 27.4 -> 28.2 mm
- net D-: track 30.0 -> 29.3 mm
- net POE: track 34.8 -> 34.3 mm
- net GND: vias 61 -> 64
Other:
- outline, holes or cut-outs redrawn
- board text added: "Ag9912-LP"
- board text added: "Designed by RevK www.me.uk"
- board text added: "Faikout PoE"
- board text removed: "Faikout"

Commit message: Latest tweaks
Parts:
- removed D21: DKS34, RevK:D_SOD-123FL
- added P2: Square, RevK:PAD-2mm, B.Cu at (135.5, 52.5)
- added P3: Square, RevK:PAD-2mm, B.Cu at (138.0, 52.5)
- added P4: Square, RevK:PAD-2mm, B.Cu at (140.5, 52.5)
- moved C22 8.29 mm to (116.6, 59.4)
- moved P1 3.20 mm to (134.0, 57.0)
Connections:
- C22 pad 1: POE -> VDC
- C25 pad 2: POE -> VDC
- C26 pad 1: POE -> VDC
- F4 pad 1: POE -> VDC
- F4 pad 2: Net-(F4-Pad2) -> POE
- M1 pad 1: Net-(F4-Pad2) -> POE
- M1 pad 2: Net-(F4-Pad2) -> POE
- R20 pad 2: POE -> VDC
- R21 pad 1: POE -> VDC
Routing:
- net VDC: track 28.2 -> 57.4 mm
- net POE: track 34.3 -> 7.86 mm
- net Net-(F4-Pad2): track 7.86 -> 0.00 mm
- net D+: track 28.2 -> 32.6 mm
- net Net-(P1-P): track 8.55 -> 6.06 mm
- net D-: track 29.3 -> 31.6 mm
Other:
- board text added: "D+"
- board text added: "D-"
- board text added: "⏚"

Commit message: Smaller design
Parts:
- J7: moved to B.Cu
- moved C36 35.0 mm to (105.6, 56.4), turned to 90 degrees
- moved R9 34.7 mm to (105.0, 56.4), turned to -90 degrees
- moved C2 32.4 mm to (128.1, 60.5), turned to 180 degrees
- moved FB4 30.3 mm to (128.2, 61.5), turned to 180 degrees
- moved C5 28.0 mm to (128.4, 62.6), turned to 180 degrees
- moved C34 26.7 mm to (128.1, 63.5), turned to -90 degrees
- moved C3 25.6 mm to (130.2, 63.4), turned to 90 degrees
- moved FB5 25.5 mm to (127.2, 64.8), turned to 90 degrees
- moved C4 25.2 mm to (130.8, 63.4), turned to 90 degrees
- moved R7 25.0 mm to (131.3, 63.4), turned to 90 degrees
- moved P1 25.0 mm to (113.0, 70.5)
- moved D2 24.7 mm to (132.1, 63.4), turned to 90 degrees
- moved C16 23.9 mm to (134.3, 63.6), turned to 0 degrees
- moved D1 22.4 mm to (133.7, 64.4), turned to 0 degrees
- moved L14 20.9 mm to (116.4, 98.0), turned to 90 degrees
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Connections:
- J1 pad S1: unconnected-(J1-PadS1) -> VIN-
- J1 pad S2: GND -> VIN-
Routing:
- net TX: track 46.3 -> 10.2 mm
- net +3.3V: track 141.5 -> 110.5 mm, vias 4 -> 2
- net SI: track 47.6 -> 16.8 mm
- net POELOAD: track 36.5 -> 6.48 mm
- net RX: track 41.3 -> 12.7 mm
- net PME: track 33.5 -> 11.9 mm
- net GND: track 20.9 -> 0.00 mm, vias 64 -> 55
- net INTR: track 33.3 -> 12.5 mm
- net SCLK: track 37.9 -> 18.4 mm
- net CSN: track 40.9 -> 21.7 mm
- net RXP: track 28.4 -> 10.1 mm
- net RXN: track 26.4 -> 9.83 mm
- net E12: track 12.7 -> 28.3 mm, vias 0 -> 2
- net TXP: track 21.5 -> 7.57 mm
- net VIN+: track 29.4 -> 15.5 mm
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Other:
- board size 42 x 69 mm -> 39 x 65 mm
- board text added: "10/100 Ethernet PoE"
- board text added: "ABE"
- board text added: "FaikoutPOE"
- board text removed: "${CURRENT_DATE}"
- board text removed: "10/100 Ethernet"
- board text removed: "AB"
- board text removed: "B"
- board text removed: "E"
- board text removed: "Faikout PoE"
