File: PCB/FaikoutPOE/Faikout.kicad_pcb (KiCad board)
At the start: 2 copper layers, 39 x 65 mm, 87 parts, among them J1 RJ45_LED, J3 S21, J5 Reset, J7 TC2030-USB-NL-DS, M1 Ag9912-LP, P1 Square, P2 Square, P3 Square, P4 Square, Q1 BSS138PS, Q2 BSS138PS, U1 KSZ8851SNL, U2 ESP32-S3-MINI-1, U3 TCMT1100, U4 TPS62933, U5 TCMT1100, Y1 Crystal_GND24

Commit message: Red PCBs
Parts:
- added P5: Square, RevK:PAD-2mm, B.Cu at (113.0, 72.0)
- added P6: Square, RevK:PAD-2mm, B.Cu at (113.0, 74.2)
- added P7: Square, RevK:PAD-2mm, B.Cu at (109.9, 69.8)
- added P8: Square, RevK:PAD-2mm, B.Cu at (109.8, 74.1)
- moved P1 0.70 mm to (113.0, 69.8)
Connections:
- U2 pad 5: unconnected-(U2-GPIO1-Pad5) -> Net-(P5-P)
- U2 pad 6: unconnected-(U2-GPIO2-Pad6) -> Net-(P6-P)
Routing:
- net Net-(P6-P): track 0.00 -> 4.37 mm, vias 0 -> 1
- net Net-(P5-P): track 0.00 -> 4.06 mm, vias 0 -> 1
- net +3.3V: track 110.5 -> 113.2 mm, vias 2 -> 3
- net Net-(P1-P): track 4.49 -> 5.56 mm
Other:
- board text added: "1"
- board text added: "2"
- board text added: "21"
- board text added: "3V3"

Commit message: Library update
Parts:
- turned D8 to -90 degrees
- turned D9 to -90 degrees
Routing:
- net E78: track 32.3 -> 23.6 mm
- net Net-(D6-A1): track 24.6 -> 18.7 mm
- net E36: track 36.7 -> 31.3 mm
- net E45: track 27.3 -> 23.1 mm
- net Net-(D6-A2): track 25.2 -> 22.4 mm
- net E12: track 28.3 -> 27.5 mm
Other:
- board text added: "POE LOAD"

Commit message: Tweak RJ45
Other:
- outline, holes or cut-outs redrawn

Commit message: New inductor
Parts:
- removed C29: 10uF 35V, RevK:C_0603
- removed C30, C32: 100nF 35V, RevK:C_0201
- removed C31: 33nF, RevK:C_0201
- removed C33: 100uF 6.3V, RevK:C_0805
- removed L13: 4.7uH, RevK:L_5x5
- removed R12: 33k, RevK:R_0201
- removed R14: 30.9k 1%, RevK:R_0201
- removed R15: 10k, RevK:R_0201
- removed U4: TPS62933, RevK:SOT-583-8
- added C18: 10uF 35V, RevK:C_0603, F.Cu at (128.4, 56.6)
- added C19: 100nF 35V, RevK:C_0201, F.Cu at (129.4, 55.6)
- added C20: 33nF, RevK:C_0201, F.Cu at (128.7, 52.4)
- added C21: 100nF 35V, RevK:C_0201, F.Cu at (129.4, 52.6)
- added C23: 100uF 6.3V, RevK:C_0805, F.Cu at (137.2, 54.1)
- added L1: 4.7uH, RevK:L_6x6, F.Cu at (133.2, 54.1)
- added R11: 33k, RevK:R_0201, F.Cu at (127.5, 54.9)
- added R23: 30.9k 1%, RevK:R_0201, F.Cu at (127.5, 52.4)
- added R24: 10k, RevK:R_0201, F.Cu at (128.1, 52.4)
- added U6: TPS62933, RevK:SOT-583-8, F.Cu at (128.9, 54.1)
- moved C17 30.6 mm to (108.3, 73.3)
Routing:
- net +3.3V: track 113.2 -> 121.2 mm
- net VDC: track 55.2 -> 54.0 mm
- net SW: track 0.00 -> 0.77 mm
- net GND: track 0.00 -> 0.77 mm, vias 55 -> 65
Other:
- outline, holes or cut-outs redrawn

Commit message: Tweaks
Routing:
- net ETHRST: track 30.3 -> 34.0 mm
- net +1V8: track 15.7 -> 18.4 mm
