File: PCB/FaikoutPOE/Faikout.kicad_sch (KiCad schematic)
At the start: 85 parts, among them J1 RJ45_LED, J2 S21, J5 Reset, J7 TC2030-USB-NL-DS, M3 Ag97012-FL, P1 Square, Q1 BSS138PS, U1 KSZ8851SNL, U2 ESP32-S3-MINI-1, U3 TCMT1100, U4 TPS62933, U5 TCMT1100, Y1 Crystal_GND24

Commit message: Started on POE
Parts:
- removed C35: 100nF, RevK:C_0201, symbol Device:C
- removed D21: DKS34, RevK:D_SOD-123FL, symbol Device:D_Schottky
- removed D5, D6, D7: XL-1615RGBC-2812B, RevK:SMD1615-Side, symbol RevK:WS2812B-1.5mm
- added D3, D5: (no value), RevK:DFN1006-2L, symbol RevK:ES05D1MC10
- added D6, D7: D, RevK:D_0402, symbol Device:D
- J1: footprint RevK:HC-WK88-H21-DKH -> RevK:RC01516; symbol RevK:HC-WK88-H21-DKH -> RevK:RC01516; MPN C48618190 -> C708636; Position Offset (none) -> 0,0.5
- R6: value 49R9 -> 10k; MPN C100141 -> C106225
Connections:
- net POE is gone; now on net VDC: C19.1, C20.2, C21.1, F3.1, R20.2, R21.1
- net +3.3V: no longer R6.1
- net GND: now also U5.3
- net LEDI: now also D4.4 (O), U2.28 (GPIO33); no longer U2.41 (GPIO45)
- net S215V: now reaches J2.1 (Pin_1)
- net S215V: now also R6.1, U5.1
- net S21RX: now reaches J2.2 (Pin_2)
- net S21RX: now also U5.2, D5.2, D6.1 (K)
- net S21TX: now reaches J2.3 (Pin_3)
- net S21TX: now also U3.4, D3.2, D7.1 (K)
- net S21GND: now reaches J2.5 (Pin_5)
- net S21GND: now also U3.3, D3.1, D5.1
- net at R6.2: now also D6.2 (A), D7.2 (A); no longer J1.9
- net at U3.1: now also R5.2
- net TX: now reaches U3.2
- net TX: now also U2.30 (GPIO48)
- net RX: now reaches U5.4
- net RX: now also U2.29 (GPIO34)
- net LEDO: now reaches U2.27 (GPIO47)
- net LEDO: now also D4.2 (I)
- net LED: no longer names the net of U2.44 (GPIO46)
- net LED: no longer D4.2 (I)
- net LED0: no longer names the net of U1.1 (LED0)
- net LED0: no longer J1.12
- net LED1: no longer names the net of U1.32 (LED1)
- net LED1: no longer J1.10
- no-connect marks 31 -> 32
Other:
- note removed: "Consider C7423280 as no hand solder"
- moved on the sheet: J2

Commit message: PoE layout, not tracked yet
Parts:
- added R10: 49R9, RevK:R_0201, symbol Device:R
Connections:
- net S21RX: now also R10.2; no longer U5.2
- new net: R10.1, U5.2
Other:
- moved on the sheet: D3, D5, D6, D7, J2, R5, R6, U3, U5

Commit message: Tweaks
Parts:
- removed D6, D7: D, RevK:D_0402, symbol Device:D
Connections:
- net S215V: no longer U5.1
- net S21GND: now also U5.2
- net S21TX: now also R6.2
- net at R10.1: now also U5.1; no longer U5.2
Other:
- moved on the sheet: D3, D5, J2, R10, R5, R6, U3, U5

Commit message: Tweak design
Parts:
- removed C19: 100nF 35V, RevK:C_0201, symbol Device:C
- removed C20: 10uF 50V, RevK:C_1206, symbol Device:C
- removed C21: 100uF 50V, Capacitor_SMD:CP_Elec_6.3x7.7, symbol Device:C_Polarized_Small
- removed C23, C24: 10nF, RevK:C_0402, symbol Device:C
- removed D3, D5: (no value), RevK:DFN1006-2L, symbol RevK:ES05D1MC10
- removed F3: 1210L150/33WR, RevK:Fuse_1210, symbol Device:Fuse_Small
- removed J2: S21, RevK:JST_EH_S5B-EH_1x05_P2.50mm_Horizontal, symbol Connector_Generic:Conn_01x05
- removed L1, L10, L11, L12, L2, L3, L4, L5, L6, L7, L8, L9: CBG201209U121T, RevK:L_0805, symbol Device:L
- removed M3: Ag97012-FL, RevK:Ag970XX-FL, symbol RevK:Ag970XX-FL
- added C22: 100nF 35V, RevK:C_0201, symbol Device:C
- added C25: 10uF 50V, RevK:C_1206, symbol Device:C
- added C26: 100uF 50V, RevK:CP_Elec_6.3x7.7, symbol Device:C_Polarized_Small
- added D11, D7: (no value), RevK:DFN1006-2L, symbol RevK:ES05D1MC10
- added D21: DKS34, RevK:D_SOD-123FL, symbol Device:D_Schottky
- added D5: D, RevK:D_0402, symbol Device:D
- added D6: SMAJ58A, RevK:D_SMA, symbol Diode:SMAJ58A
- added D8, D9: MB4S, RevK:TO-269AA-BR, symbol Diode_Bridge:MB4S
- added F4: 1210L150/33WR, RevK:Fuse_1210, symbol Device:Fuse_Small
- added J3: S21, RevK:JST_EH_S5B-EH_1x05_P2.50mm_Horizontal, symbol Connector_Generic:Conn_01x05
- added L14, L15, L16, L17, L18, L19: CBG201209U121T, RevK:L_0805, symbol Device:L
- added M1: Ag9912-LP, RevK:Ag9900-LP, symbol RevK:Ag9912-LP_1
- added Q2: BSS138PS, RevK:SOT-363_SC-70-6, symbol RevK:BSS138PS
- added R13, R16: 10k, RevK:R_0201, symbol Device:R
- R10: value 49R9 -> 1k; MPN C100141 -> (none)
Connections:
- net S21RX is gone; now on an unnamed net: R10.2
- net E12: now also D9.2
- net E36: now also D9.1
- net E45: now also D8.2
- net E78: now also D8.1
- net GND: now also C22.2, C25.1, C26.2, M1.3 (-VDC)
- net S21GND: now also D11.2, D7.1, J3.5 (Pin_5), Q2.1 (SN), Q2.4 (DP); no longer U5.2
- net VDC: now also D21.1 (K); no longer R20.2, R21.1
- net at U5.1: no longer R10.1
- net S215V renamed S21DC
- net S21DC: now also R10.1, J3.4 (Pin_4)
- net S21TX: no longer names the net of R6.2, U3.4
- net S21TX: now also Q2.5 (GP)
- new net: D5.2 (A), J3.1 (Pin_1), R13.1
- new net: D7.2, J3.3 (Pin_3), Q2.3 (SP), R13.2
- new net: D5.1 (K), R16.1
- new net: D11.1, J3.2 (Pin_2), Q2.2 (GN), R16.2
- new net: Q2.6 (DN), U5.2
- new net: D6.2 (A2), D8.4 (-), D9.4 (-), L15.1
- new net: L15.2, L17.1
- new net: D6.1 (A1), D8.3 (+), D9.3 (+), L14.1
- new net: F4.2, M1.1 (+VDC), M1.2 (+VDC)
- new net: L17.2, L19.1
- new net: L14.2, L16.1
- new net: L16.2, L18.1
- new net POE: C22.1, C25.2, C26.1, D21.2 (A), F4.1, R20.2, R21.1
- new net VIN+: L18.2, M1.5 (VIN+), M1.6 (VIN+)
- new net VIN-: L19.2, M1.7 (VIN-), M1.8 (VIN-)
- no-connect marks 32 -> 29
Other:
- moved on the sheet: C11, C34, D4, J1, R5, R6, TR1, U3, U5

Commit message: Started POE
Parts:
- Y1: footprint Crystal:Crystal_SMD_3225-4Pin_3.2x2.5mm -> RevK:Crystal-3.2x2.5
Connections:
- net VBUS is gone; now on net VDC: J7.1 (VBUS)
- net GND: now also J1.S2
- no-connect marks 29 -> 30

Commit message: More tracking
Parts:
- M1: now left out of the parts list
Changed lines of the file:
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@@
 		(body_style 1)
 		(exclude_from_sim no)
-		(in_bom yes)
+		(in_bom no)
 		(on_board yes)
-		(in_pos_files yes)
+		(in_pos_files no)
 		(dnp no)
 		(fields_autoplaced yes)
