File: PCB/FaikoutPOE/Faikout.kicad_sch (KiCad schematic)
At the start: 83 parts, among them J1 RJ45_LED, J3 S21, J5 Reset, J7 TC2030-USB-NL-DS, M1 Ag9912-LP, P1 Square, Q1 BSS138PS, Q2 BSS138PS, U1 KSZ8851SNL, U2 ESP32-S3-MINI-1, U3 TCMT1100, U4 TPS62933, U5 TCMT1100, Y1 Crystal_GND24

Commit message: Finished PoE
Parts:
- D8, D9: MPN (none) -> C232847
- U3: MPN (none) -> C118298; Rotation Offset (none) -> 90
- U5: MPN (none) -> MPN; Rotation Offset (none) -> 90
Changed lines of the file:
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@@
 			)
 		)
+		(property "MPN" "C232847"
+			(at 33.02 181.61 90)
+			(hide yes)
+			(show_name no)
+			(do_not_autoplace no)
+			(effects
+				(font
+					(size 1.27 1.27)
+				)
+			)
+		)
 		(pin "4"
 		)
@@
 			)
 		)
+		(property "MPN" "C118298"
+			(at 201.93 121.92 0)
+			(hide yes)
+			(show_name no)
+			(do_not_autoplace no)
+			(effects
+				(font
+					(size 1.27 1.27)
+				)
+			)
+		)
+		(property "Rotation Offset" "90"
+			(at 201.93 121.92 0)
+			(hide yes)
+			(show_name no)
+			(do_not_autoplace no)
+			(effects
+				(font
+					(size 1.27 1.27)
+				)
+			)
+		)
 		(pin "1"
 		)
@@
 			)
 		)
+		(property "MPN" "MPN"
+			(at 201.93 135.89 0)
+			(hide yes)
+			(show_name no)
+			(do_not_autoplace no)
+			(effects
+				(font
+					(size 1.27 1.27)
+				)
+			)
+		)
+		(property "Rotation Offset" "90"
+			(at 201.93 135.89 0)
+			(hide yes)
+			(show_name no)
+			(do_not_autoplace no)
+			(effects
+				(font
+					(size 1.27 1.27)
+				)
+			)
+		)
 		(pin "1"
 		)
@@
 			(hide yes)
 			(show_name no)
+			(do_not_autoplace no)
+			(effects
+				(font
+					(size 1.27 1.27)
+				)
+			)
+		)
+		(property "MPN" "C232847"
+			(at 52.07 181.61 90)
+			(hide yes)
+			(show_name no)

Commit message: Tidy tracks
Parts:
- U1: Rotation Offset 90 -> -90
Changed lines of the file:
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@@
 			)
 		)
-		(property "Rotation Offset" "90"
+		(property "Rotation Offset" "-90"
 			(at 66.04 66.04 0)
 			(hide yes)
