File: PCB/FaikoutPOE/Faikout.kicad_sch (KiCad schematic)
At the start: 83 parts, among them J1 RJ45_LED, J3 S21, J5 Reset, J7 TC2030-USB-NL-DS, M1 Ag9912-LP, P1 Square, Q1 BSS138PS, Q2 BSS138PS, U1 KSZ8851SNL, U2 ESP32-S3-MINI-1, U3 TCMT1100, U4 TPS62933, U5 TCMT1100, Y1 Crystal_GND24

Commit message: Tweak
Parts:
- added D10: D, RevK:D_0402, symbol Device:D
Connections:
- net at D5.2 (A), J3.1 (Pin_1): now also D10.2 (A); no longer R13.1
- new net: D10.1 (K), R13.1
Other:
- moved on the sheet: D11, D5, D7, Q2A, Q2B, R13, R16

Commit message: Tidy
Parts:
- added R17: 1k, RevK:R_0201, symbol Device:R
- R20: value 220 1W -> 200 1W; MPN C38808 -> C2907575
Connections:
- net +3.3V: now also R17.1
- net RX: now also R17.2
Other:
- moved on the sheet: R10, R5, R6, U3, U5

Commit message: Re-render, latest layout
Parts:
- R10, R17: MPN (none) -> C270365
Changed lines of the file:
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@@
 			)
 		)
+		(property "MPN" "C270365"
+			(at 190.5 134.62 90)
+			(hide yes)
+			(show_name no)
+			(do_not_autoplace no)
+			(effects
+				(font
+					(size 1.27 1.27)
+				)
+			)
+		)
 		(pin "1"
 		)
@@
 			(hide yes)
 			(show_name no)
+			(do_not_autoplace no)
+			(effects
+				(font
+					(size 1.27 1.27)
+				)
+			)
+		)
+		(property "MPN" "C270365"
+			(at 213.36 134.62 90)
+			(hide yes)
+			(show_name no)

Commit message: Fix BOM
Parts:
- R18, R19: MPN C7467262 -> C138135
- R9: MPN C102690 -> C106225
Changed lines of the file:
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@@
 			)
 		)
-		(property "MPN" "C7467262"
+		(property "MPN" "C138135"
 			(at 31.75 58.42 90)
 			(hide yes)
@@
 			)
 		)
-		(property "MPN" "C7467262"
+		(property "MPN" "C138135"
 			(at 25.4 58.42 90)
 			(hide yes)
@@
 		(in_bom no)
 		(on_board yes)
-		(in_pos_files yes)
+		(in_pos_files no)
 		(dnp no)
 		(fields_autoplaced yes)
@@
 			)
 		)
-		(property "MPN" "C102690"
+		(property "MPN" "C106225"
 			(at 274.32 76.2 90)
 			(hide yes)

Commit message: Latest tweaks
Parts:
- removed D21: DKS34, RevK:D_SOD-123FL, symbol Device:D_Schottky
- added P2, P3, P4: Square, RevK:PAD-2mm, symbol RevK:Square
Connections:
- net D+: now also P3.1 (P)
- net D-: now also P2.1 (P)
- net GND: now also P4.1 (P)
- net POE: now also F4.2, M1.1 (+VDC), M1.2 (+VDC); no longer C22.1, C25.2, C26.1, F4.1, R20.2, R21.1
- net VDC: now also C22.1, C25.2, C26.1, F4.1, R20.2, R21.1
Other:
- moved on the sheet: F4, Q1A, Q1B, R20, R21, R22

Commit message: Smaller design
Connections:
- net GND: no longer J1.S2
- net VIN-: now also J1.S1, J1.S2
- no-connect marks 30 -> 29
Other:
- moved on the sheet: C11, J1, TR1

Commit message: Extra GPIOs
Parts:
- U1: footprint RevK:QFN-32-1EP_5x5mm_P0.5mm_EP3.7x3.7mm -> RevK:QFN-32-1EP_5x5mm_P0.5mm_EP3.7x3.7mm-hot
Connections:
- net VIN-: now also J1.S; no longer J1.S1, J1.S2
Changed lines of the file:
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@@
 	)
 	(junction
-		(at 17.78 165.1)
-		(diameter 0)
-		(color 0 0 0 0)
-	)
-	(junction
 		(at 40.64 105.41)
 		(diameter 0)
@@
 	(wire
 		(pts
-			(xy 33.02 137.16) (xy 17.78 137.16)
-		)
-		(stroke
-			(width 0)
-			(type default)
-		)
-	)
-	(wire
-		(pts
 			(xy 88.9 30.48) (xy 92.71 30.48)
 		)
@@
 	(wire
 		(pts
-			(xy 17.78 137.16) (xy 17.78 165.1)
-		)
-		(stroke
-			(width 0)
-			(type default)
-		)
-	)
-	(wire
-		(pts
 			(xy 76.2 30.48) (xy 76.2 44.45)
 		)
@@
 			)
 		)
-		(property "Footprint" "RevK:QFN-32-1EP_5x5mm_P0.5mm_EP3.7x3.7mm"
+		(property "Footprint" "RevK:QFN-32-1EP_5x5mm_P0.5mm_EP3.7x3.7mm-hot"
 			(at 65.786 30.988 0)
 			(hide yes)
@@
 		(pin "4"
 		)
-		(pin "S1"
-		)
-		(pin "S2"
+		(pin "S"
 		)
 		(instances

Commit message: Red PCBs
Parts:
- added P5, P6, P7, P8: Square, RevK:PAD-2mm, symbol RevK:Square
Connections:
- net +3.3V: now also P7.1 (P)
- net GND: now also P8.1 (P)
- net at U2.5 (GPIO1): now also P5.1 (P)
- net at U2.6 (GPIO2): now also P6.1 (P)
- no-connect marks 29 -> 27
Other:
- moved on the sheet: C17
