File: PCB/Faikout/Faikout.kicad_pcb (KiCad board)
At the start: 2 copper layers, 70 x 70 mm, 41 parts, among them J1 S21, J2 TC2030-USB-NL, J3 Reset, Q1 BSS138PS, U4 ESP32-S3-MINI-1, U5 TPS62933

Commit message: OSP ordered
Other:
- board text added: "OSP"

Commit message: Extra GPIOs
Parts:
- added TP11: TestPoint, RevK:PAD-2mm, B.Cu at (125.2, 67.4)
- added TP12: TestPoint, RevK:PAD-2mm, B.Cu at (125.2, 65.0)
- added TP13: TestPoint, RevK:PAD-2mm, B.Cu at (125.2, 62.6)
- moved TP6 4.50 mm to (130.9, 60.3)
- moved TP8 4.50 mm to (126.4, 60.2)
- moved J3 1.75 mm to (131.5, 65.0)
- moved L13 0.20 mm to (141.2, 70.0)
Connections:
- U4 pad 4: unconnected-(U4-GPIO0-Pad4) -> Net-(U4-GPIO0)
- U4 pad 5: unconnected-(U4-GPIO1-Pad5) -> Net-(U4-GPIO1)
- U4 pad 6: unconnected-(U4-GPIO2-Pad6) -> Net-(U4-GPIO2)
Routing:
- net Net-(U4-GPIO2): track 0.00 -> 10.6 mm, vias 0 -> 1
- net Net-(U4-GPIO1): track 0.00 -> 7.83 mm, vias 0 -> 1
- net Net-(U4-GPIO0): track 0.00 -> 5.12 mm, vias 0 -> 1
- net +3.3V: track 50.8 -> 53.3 mm
- net Net-(J3-Pin_2): track 7.10 -> 5.35 mm
- net D-: track 37.0 -> 35.8 mm
- net GND: track 5.63 -> 4.66 mm, vias 91 -> 94
- net RST: track 20.3 -> 19.3 mm
- net TX: track 5.41 -> 6.03 mm
- net D+: track 41.8 -> 42.3 mm
Other:
- board text added: "0"
- board text added: "2"
- board text removed: "OSP"
