File: PCB/Faikout/Faikout.kicad_sch (KiCad schematic)
At the start: 41 parts, among them J1 S21, J2 TC2030-USB-NL, J3 Reset, Q1 BSS138PS, U4 ESP32-S3-MINI-1, U5 TPS62933

Commit message: Extra GPIOs
Parts:
- added TP11, TP12, TP13: TestPoint, RevK:PAD-2mm, symbol Connector:TestPoint
Connections:
- net at U4.4 (GPIO0): now also TP11.1
- net at U4.5 (GPIO1): now also TP12.1
- net at U4.6 (GPIO2): now also TP13.1
- no-connect marks 25 -> 22
Other:
- moved on the sheet: C6, FID2, FID3, J3, R3, U4
